Commit message: add joint group state default.

File: interbotix_ros_xsarms/interbotix_xsarm_moveit/config/srdf/vx300s.srdf.xacro (robot description, xacro)
@@ -55,4 +55,12 @@
         <joint name="wrist_angle" value="0.8" />
         <joint name="wrist_rotate" value="0" />
+    </group_state>
+    <group_state name="Default" group="interbotix_arm">
+        <joint name="waist" value="0.0" />
+        <joint name="shoulder" value="-0.5" />
+        <joint name="elbow" value="0.5" />
+        <joint name="forearm_roll" value="0" />
+        <joint name="wrist_angle" value="-0.3" />
+        <joint name="wrist_rotate" value="0.0" />
     </group_state>
     <group_state name="Grasping" group="interbotix_gripper">

Commit message: Update group position , upte rivze

File: interbotix_ros_xsarms/interbotix_xsarm_moveit/config/srdf/vx300s.srdf.xacro (robot description, xacro)
@@ -58,8 +58,8 @@
     <group_state name="Default" group="interbotix_arm">
         <joint name="waist" value="0.0" />
-        <joint name="shoulder" value="-0.5" />
-        <joint name="elbow" value="0.5" />
+        <joint name="shoulder" value="-1.0472" />
+        <joint name="elbow" value="0.35" />
         <joint name="forearm_roll" value="0" />
-        <joint name="wrist_angle" value="-0.3" />
+        <joint name="wrist_angle" value="1.22" />
         <joint name="wrist_rotate" value="0.0" />
     </group_state>

Commit message: modify default pose

File: interbotix_ros_xsarms/interbotix_xsarm_moveit/config/srdf/vx300s.srdf.xacro (robot description, xacro)
@@ -58,8 +58,8 @@
     <group_state name="Default" group="interbotix_arm">
         <joint name="waist" value="0.0" />
-        <joint name="shoulder" value="-1.0472" />
+        <joint name="shoulder" value="-1.05" />
         <joint name="elbow" value="0.35" />
         <joint name="forearm_roll" value="0" />
-        <joint name="wrist_angle" value="1.22" />
+        <joint name="wrist_angle" value="1.25" />
         <joint name="wrist_rotate" value="0.0" />
     </group_state>

Commit message: Update Default pose

File: interbotix_ros_xsarms/interbotix_xsarm_moveit/config/srdf/vx300s.srdf.xacro (robot description, xacro)
@@ -61,5 +61,5 @@
         <joint name="elbow" value="0.35" />
         <joint name="forearm_roll" value="0" />
-        <joint name="wrist_angle" value="1.25" />
+        <joint name="wrist_angle" value="1.05" />
         <joint name="wrist_rotate" value="0.0" />
     </group_state>
